File: ATMEL-ICE-Octopus-Back/ATMEL-ICE-Octopus-Back.kicad_pcb (KiCad board)
At the start: 2 copper layers, 10 x 40 mm, 5 parts, among them J1 ATMEL-ICE SAM SOCKET, J2 ATMEL-ICE AVR SOCKET, J3 Angled Conn 1, J4 Angled Conn 2, J5 Angled Conn 3

Commit message: ATMEL-ICE-Octopus-Back: rev A1 - add OHL license and use kibot
Other:
- board text added: "${license}"
- board text added: "rev ${rev}"
- board text removed: "rev A0"
Changed lines of the file:
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@@
   )
   (paper "A4")
+  (title_block
+    (rev "${rev}")
+  )
   (layers
     (0 "F.Cu" signal)
@@
     )
   )
+  (property "license" "Licensed under CERN-OHL-W v2")
+  (property "rev" "A1")
   (net 0 "")
   (net 1 "/VTG")
@@
   (gr_arc (start 100 81) (mid 100.292893 80.292893) (end 101 80) (layer "Edge.Cuts") (width 0.1))
   (gr_arc (start 101 120) (mid 100.292894 119.707106) (end 100 119) (layer "Edge.Cuts") (width 0.1))
+  (gr_text "${license}" (at 108.51 100.05 -90) (layer "B.SilkS")
+    (effects (font (size 1 1) (thickness 0.154)) (justify mirror))
+  )
   (gr_text "JLCJLCJLCJLC" (at 108.7 92.1 90) (layer "F.SilkS")
     (effects (font (size 1.1 1.1) (thickness 0.154)))
   )
-  (gr_text "rev A0" (at 108.6 105.4 90) (layer "F.SilkS")
+  (gr_text "rev ${rev}" (at 108.6 105.4 90) (layer "F.SilkS")
     (effects (font (size 1.3 1.3) (thickness 0.18)) (justify right))
   )
