File: ATMEL-ICE-Octopus/ATMEL-ICE-Octopus.kicad_sch (KiCad schematic)
At the start: 75 parts, among them J1 ATMEL-ICE SAM SOCKET, J11 ARM Multi-ICE 20-pin JTAG, J12 SWD/JTAG SAM (ARM/Cortex-M db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, J13 SWD/JTAG AVR, J14 aWire/(U)PDI/TPI/debugWire/SP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, J15 SWD, J16 Conn_01x01_Female, J2 ATMEL-ICE AVR SOCKET, J21 Conn_01x03, J22 Conn_01x03, J23 Conn_01x03, J24 Conn_01x03, J3 Angled Conn 1, J4 Angled Conn 2, J5 Angled Conn 3, J8 Conn_01x01_Female, J9 Conn_01x03, Q13 BC846, Q14 BC846, Q15 BC846, Q17 BC846, Q19 Q_PMOS_FDV304P, Q23 BC846, Q24 BC846, Q25 BC846, Q27 BC846, Q29 Q_PMOS_FDV304P, U11 SGM708, U12 TPS2049D, U21 SGM708, U22 TPS2049D

Commit message: ATMEL-ICE-Octopus: rev B5
Parts:
- removed D11, D26: GREEN, LED_SMD:LED_0805_2012Metric_Pad1.15x1.40mm_HandSolder, symbol Device:LED_Small
- removed D12, D28: RED, LED_SMD:LED_0805_2012Metric_Pad1.15x1.40mm_HandSolder, symbol Device:LED_Small
- removed D19, D29: BAT48ZFILM, AA-OSA-Packages:D_MiniMELF, symbol Diode:BAT48ZFILM
- removed J16: Conn_01x01_Female, Connector_PinSocket_2.54mm:PinSocket_1x02_P2.54mm_Vertical, symbol Connector:Conn_01x02_Female
- removed J21, J22, J23, J24, J9: Conn_01x03, Connector_PinHeader_2.54mm:PinHeader_1x03_P2.54mm_Vertical, symbol Connector_Generic:Conn_01x03
- removed J3: Angled Conn 1, AA-OSA-connectors:PinHeader_2x02_P2.54mm_Vertical_NoSilk, symbol Connector_Generic:Conn_02x02_Odd_Even
- removed J4: Angled Conn 2, AA-OSA-connectors:PinHeader_2x02_P2.54mm_Vertical_NoSilk, symbol Connector_Generic:Conn_02x02_Odd_Even
- removed J5: Angled Conn 3, AA-OSA-connectors:PinHeader_2x02_P2.54mm_Vertical_NoSilk, symbol Connector_Generic:Conn_02x02_Odd_Even
- removed JP1, JP2: Jumper_2_Open, Connector_PinHeader_2.54mm:PinHeader_2x01_P2.54mm_Vertical, symbol Jumper:Jumper_2_Open
- removed Q13, Q14, Q15, Q17, Q23, Q24, Q25, Q27: BC846, Package_TO_SOT_SMD:SOT-23, symbol Transistor_BJT:BC846
- removed Q19, Q29: Q_PMOS_FDV304P, Package_TO_SOT_SMD:SOT-23, symbol AA-OSA-Basic:Q_PMOS_FDV304P
- removed R11, R12, R21, R22: 100k, Resistor_SMD:R_0805_2012Metric_Pad1.20x1.40mm_HandSolder, symbol Device:R
- removed R13, R14, R19, R23, R24, R29: 47k, Resistor_SMD:R_0805_2012Metric_Pad1.20x1.40mm_HandSolder, symbol Device:R
- removed R15, R17, R25, R27, R34, R44: 22k, Resistor_SMD:R_0805_2012Metric_Pad1.20x1.40mm_HandSolder, symbol Device:R
- removed R16, R18, R26, R28: 1k, Resistor_SMD:R_0805_2012Metric_Pad1.20x1.40mm_HandSolder, symbol Device:R
- removed R31, R41: 12k, Resistor_SMD:R_0805_2012Metric_Pad1.20x1.40mm_HandSolder, symbol Device:R
- removed R32, R35, R42, R45: 470, Resistor_SMD:R_0805_2012Metric_Pad1.20x1.40mm_HandSolder, symbol Device:R
- removed R33, R36, R43, R46: 28, Resistor_SMD:R_0805_2012Metric_Pad1.20x1.40mm_HandSolder, symbol Device:R
- removed R37, R47: 18k, Resistor_SMD:R_0805_2012Metric_Pad1.20x1.40mm_HandSolder, symbol Device:R
- removed R38, R48: 1.8k, Resistor_SMD:R_0805_2012Metric_Pad1.20x1.40mm_HandSolder, symbol Device:R
- removed R39, R49: 220, Resistor_SMD:R_0805_2012Metric_Pad1.20x1.40mm_HandSolder, symbol Device:R
- removed U11, U21: SGM708, AA-OSA-Packages:SO-8_3.9x4.9mm_P1.27mm, symbol AA-OSA-Power:SGM708
- removed U12, U22: TPS2049D, AA-OSA-Packages:SO-8_3.9x4.9mm_P1.27mm, symbol AA-OSA-Power:TPS2049D
- added D1: SMAJ13A, AA-OSA-Packages:D_SMA+SMP_Handsoldering, symbol Device:D
- added H1, H2, H3: MountingHole, MountingHole:MountingHole_2.5mm, symbol Mechanical:MountingHole
- added J16: conn_01x01, Connector_PinHeader_2.54mm:PinHeader_1x01_P2.54mm_Vertical, symbol Connector_Generic:Conn_01x01
- added J17: Conn_01x02_Female, Connector_PinSocket_2.54mm:PinSocket_1x02_P2.54mm_Vertical, symbol Connector:Conn_01x02_Female
- added J18: conn_02x03_Female, Connector_PinSocket_2.54mm:PinSocket_2x03_P2.54mm_Vertical, symbol Connector_Generic:Conn_02x03_Odd_Even
- added J21, J23: Conn_01x02_Angled, Connector_PinHeader_2.00mm:PinHeader_1x02_P2.00mm_Horizontal, symbol Connector_Generic:Conn_01x02
- added J22: Conn_02x02_Angled, Connector_PinHeader_2.00mm:PinHeader_2x02_P2.00mm_Horizontal, symbol Connector_Generic:Conn_01x04
- added J31, J33: Conn_01x02_Angled, AA-OSA-connectors:PinHeader_1x02_P2.00mm_Angled, symbol Connector_Generic:Conn_01x02
- added J32: Conn_02x02_Angled, AA-OSA-connectors:PinHeader_2x02_P2.00mm_Angled, symbol Connector_Generic:Conn_01x04
- added J8: ~, AA-OSA-connectors:PinHeader_2x03_P2.54mm_Horizontal_Jumper, symbol Connector_Generic:Conn_02x03_Odd_Even
- added MB1, MB2, MB3, MB4: Mouse bites, AA-OSA-misc:mouse-bite-3x4mm-slot, symbol Mechanical:MountingHole
- J1: value ATMEL-ICE SAM SOCKET -> conn_02x05
- J11: value ARM Multi-ICE 20-pin JTAG -> conn_02x10
- J12: value SWD/JTAG SAM (ARM/Cortex-M dbg) -> conn_02x05_key7
- J13: value SWD/JTAG AVR -> conn_02x05_key7
- J14: value aWire/(U)PDI/TPI/debugWire/SPI Target -> conn_02x03
- J15: value SWD -> conn_01x04
- J2: value ATMEL-ICE AVR SOCKET -> conn_02x05
- J6: renamed from J8; footprint Connector_PinSocket_2.54mm:PinSocket_1x02_P2.54mm_Vertical -> Connector_PinSocket_2.54mm:PinSocket_1x01_P2.54mm_Vertical; symbol Connector:Conn_01x02_Female -> Connector:Conn_01x01_Female
Connections:
- net VIN2 is gone; now on net VIN_JTAG: J12.1 (Pin_1)
- net VIN3 is gone; now on net VIN_JTAG: J13.4 (Pin_4)
- net GND: now also D1.2 (A), J17.2 (Pin_2), J21.1 (Pin_1), J31.1 (Pin_1); no longer J6.1 (Pin_1)
- net TCK: now also J18.3 (Pin_3), J22.3 (Pin_3), J32.3 (Pin_3)
- net TDI: now also J18.1 (Pin_1), J22.1 (Pin_1), J32.1 (Pin_1)
- net TDO: now also J18.2 (Pin_2), J22.2 (Pin_2), J32.2 (Pin_2)
- net TMS: now also J18.4 (Pin_4), J22.4 (Pin_4), J32.4 (Pin_4)
- net VTG: now also J6.1 (Pin_1), J21.2 (Pin_2), J31.2 (Pin_2); no longer J6.2 (Pin_2)
- net nSRST: now also J18.5 (Pin_5), J23.2 (Pin_2), J33.2 (Pin_2)
- net nTRST: now also J18.6 (Pin_6), J23.1 (Pin_1), J33.1 (Pin_1)
- net VIN1 renamed VIN_JTAG
- net VIN_JTAG: now also J8.3 (Pin_3)
- net VIN4 renamed VIN_AVR
- net VIN_AVR: now also J8.1 (Pin_1)
- new net VIN: D1.1 (K), J8.2 (Pin_2), J8.4 (Pin_4), J8.6 (Pin_6)
- new net VIN_PROBE: J16.1 (Pin_1), J17.1 (Pin_1), J8.5 (Pin_5)
- no-connect marks 19 -> 10
Other:
- added sheet StatusLeds (StatusLeds.kicad_sch)
- added sheet VoltageBooster (VoltageBooster.kicad_sch)
- added sheet VoltageLimiter (VoltageLimiter.kicad_sch)
- note added: "6-PIN VARIOUS: AVR aWire AVR SPI + debugWire AVR (U)PDI AVR TPI"
- note added: "ARDUINO 4-PIN DEBUG CONNECTOR with added VCC"
- note added: "ATMEL-ICE AVR SOCKET"
- note added: "ATMEL-ICE SAM SOCKET"
- note added: "JTAG/SWD SAM (ARM/Cortex-M dbg)"
- note removed: "6-PIN VARIOUS"
- note removed: "ARDUINO 4-PIN DEBUG CONNECTOR"
- note removed: "ARM JTAG (10-pin standard)"
- note removed: "AVR JTAG"
- note removed: "Bypass of onboard power management (dangerous)"
- note removed: "INPUT VOLTAGE SENSING"
- note removed: "NB : must use VCCIO probe as well."
- note removed: "POWER PATH SWITCHING"
- note removed: "Select 3.5V or 5.5V VCCIO limit"
- note removed: "Takes VTG (Target I/O Reference Voltage) from either the RED (VCCIO probe) if present, BLACK (Target Connectors) otherwise. Turns on VTG only if input voltage is above ~3V and below the limit as set by LIMIT_LOW jumper and divider networks."
- note removed: "USE_BLACK asserted (1) when: - VDD_BLACK > 2.93V - BLACK_SENSE < 1.25V - VDD_RED < 0.6V - 200ms until all above conditions are met"
- note removed: "USE_RED asserted (1) when: - VDD_RED> 2.93V - RED_SENSE < 1.25V - USE_BLACK low (< 0.6V) - 200ms until all above conditions are met"
- note removed: "VCCIO PROBE"
- moved on the sheet: J13, J14, J15

Commit message: ATMEL-ICE-Octopus: rev B6
Parts:
- added JP1, JP2: SolderJumper_3_Bridged12, Jumper:SolderJumper-3_P1.3mm_Bridged2Bar12_RoundedPad1.0x1.5mm_NumberLabels, symbol Jumper:SolderJumper_3_Bridged12
- added R56: 1M, Resistor_SMD:R_0805_2012Metric_Pad1.20x1.40mm_HandSolder, symbol Device:R
Connections:
- net GND: now also R56.1
- net VIN: now also JP1.3 (B), JP2.3 (B)
- net VLED: now also JP2.2 (C)
- net VTG: now also JP1.2 (C), R56.2
- new net VoltageBooster/VBOOST: JP2.1 (A)
- new net VoltageLimiter/VOUT: JP1.1 (A)
Other:
- sheet VoltageBooster ports: added VBOOST; removed VLED
- moved on the sheet: D1, J8
