File: ATMEL-ICE-Octopus/VoltageBooster.kicad_sch (KiCad schematic)
At the start: 22 parts, among them Q61 CPH3910, Q62 NXV100XP, Q63 BC857B, U71 AP3015A

Commit message: ATMEL-ICE-Octopus: rev B6
Connections:
- net VLED renamed VBOOST
Changed lines of the file:
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@@
     (effects (font (size 1.27 1.27)) (justify left bottom))
   )
-  (label "VLED" (at 241.3 31.75 0)
+  (label "VBOOST" (at 237.49 31.75 0)
     (effects (font (size 1.27 1.27)) (justify left bottom))
   )
@@
     (effects (font (size 1.27 1.27)) (justify right))
   )
-  (hierarchical_label "VLED" (shape output) (at 259.08 31.75 0)
+  (hierarchical_label "VBOOST" (shape output) (at 259.08 31.75 0)
     (effects (font (size 1.27 1.27)) (justify left))
   )
